File: eBoard_remote_control/eBoard_remote_control.sch (KiCad schematic (older format))
At the start: 38 parts, among them J1 SWDIO_conn, P1 USB, U1 MDBT42, U2 AP2112(3.3V), U3 MCP73831T-2ACI/OT, U4 CP2104, U5 AH49ENTR-G1, U6 AH49ENTR-G1, U7 AH49ENTR-G1, X2 JSTPH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

Commit message: V2 update
Parts:
- removed J1: SWDIO_conn, Connector_PinHeader_2.54mm:PinHeader_1x05_P2.54mm_Vertical, symbol Connector:Conn_01x05_Male
- added C9: 0.1uF, eBoard_remote_control:C0603, symbol eBoard_remote_control-eagle-import:CAP_CERAMIC0603_NO
- added D4: 1n4148, Adafruit nRF52 Bluefruit Feather rev G:SOD-323, symbol eBoard_remote_control-eagle-import:DIODESOD-323
- added J1: SWDIO_conn, Connector_PinHeader_1.27mm:PinHeader_2x05_P1.27mm_Vertical_SMD, symbol Adafruit_nRF52_Bluefruit_Feather_rev_G-cache:Adafruit_nRF52_Bluefruit_Feather_r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
- added R2: 10K, eBoard_remote_control:0603-NO, symbol eBoard_remote_control-eagle-import:RESISTOR0805_NOOUTLINE
- added SJ2: BAT, Adafruit nRF52 Bluefruit Feather rev G:SOLDERJUMPER_CLOSEDWIRE, symbol eBoard_remote_control-eagle-import:SOLDERJUMPERCLOSED
- C1, C10, C12, C2, C4: footprint eBoard_remote_control:0603-NO -> eBoard_remote_control:C0603
- C3, C5, C6, C7, C8: footprint eBoard_remote_control:0805-NO -> eBoard_remote_control:C0603
- DIS1: footprint Connector_PinHeader_2.54mm:PinHeader_1x04_P2.54mm_Vertical -> eBoard_remote_control:OLED
Connections:
- wire segments 170 -> 188
Changed lines of the file:
@@
 F 0 "C1" V 3109 9949 50  0000 C CNN
 F 1 "22pF" V 3290 9949 50  0000 C CNN
-F 2 "eBoard_remote_control:0603-NO" H 3200 9900 50  0001 C CNN
+F 2 "eBoard_remote_control:C0603" H 3200 9900 50  0001 C CNN
 F 3 "" H 3200 9900 50  0001 C CNN
 	1    3200 9900
@@
 F 0 "C2" V 3709 9949 50  0000 C CNN
 F 1 "22pF" V 3890 9949 50  0000 C CNN
-F 2 "eBoard_remote_control:0603-NO" H 3800 9900 50  0001 C CNN
+F 2 "eBoard_remote_control:C0603" H 3800 9900 50  0001 C CNN
 F 3 "" H 3800 9900 50  0001 C CNN
 	1    3800 9900
@@
 F 0 "C3" V 2909 8649 50  0000 C CNN
 F 1 "10uF" V 3090 8649 50  0000 C CNN
-F 2 "eBoard_remote_control:0805-NO" H 3000 8600 50  0001 C CNN
+F 2 "eBoard_remote_control:C0603" H 3000 8600 50  0001 C CNN
 F 3 "" H 3000 8600 50  0001 C CNN
 	1    3000 8600
@@
 F 0 "C4" V 2009 8549 50  0000 C CNN
 F 1 "1uF" V 2190 8549 50  0000 C CNN
-F 2 "eBoard_remote_control:0603-NO" H 2100 8500 50  0001 C CNN
+F 2 "eBoard_remote_control:C0603" H 2100 8500 50  0001 C CNN
 F 3 "" H 2100 8500 50  0001 C CNN
 	1    2100 8500
@@
 F 0 "C5" V 5009 2449 50  0000 C CNN
 F 1 "10µF" V 5190 2449 50  0000 C CNN
-F 2 "eBoard_remote_control:0805-NO" H 5100 2400 50  0001 C CNN
+F 2 "eBoard_remote_control:C0603" H 5100 2400 50  0001 C CNN
 F 3 "" H 5100 2400 50  0001 C CNN
 	1    5100 2400
@@
 F 0 "C6" V 2309 4649 50  0000 C CNN
 F 1 "10µF" V 2490 4649 50  0000 C CNN
-F 2 "eBoard_remote_control:0805-NO" H 2400 4600 50  0001 C CNN
+F 2 "eBoard_remote_control:C0603" H 2400 4600 50  0001 C CNN
 F 3 "" H 2400 4600 50  0001 C CNN
 	1    2400 4600
@@
 F 0 "C8" V 3909 4649 50  0000 C CNN
 F 1 "10µF" V 4090 4649 50  0000 C CNN
-F 2 "eBoard_remote_control:0805-NO" H 4000 4600 50  0001 C CNN
+F 2 "eBoard_remote_control:C0603" H 4000 4600 50  0001 C CNN
 F 3 "" H 4000 4600 50  0001 C CNN
 	1    4000 4600
@@
 F 0 "C10" V 10409 6949 50  0000 C CNN
 F 1 "0.1uF" V 10590 6949 50  0000 C CNN
-F 2 "eBoard_remote_control:0603-NO" H 10500 6900 50  0001 C CNN
+F 2 "eBoard_remote_control:C0603" H 10500 6900 50  0001 C CNN
 F 3 "" H 10500 6900 50  0001 C CNN
 	1    10500 6900
@@
 F 0 "C12" V 5309 4649 50  0000 C CNN
 F 1 "1nF" V 5490 4649 50  0000 C CNN
-F 2 "eBoard_remote_control:0603-NO" H 5400 4600 50  0001 C CNN
+F 2 "eBoard_remote_control:C0603" H 5400 4600 50  0001 C CNN
 F 3 "" H 5400 4600 50  0001 C CNN
 	1    5400 4600
@@
 F 0 "C7" V 10609 8249 50  0000 C CNN
 F 1 "10uf" V 10790 8249 50  0000 C CNN
-F 2 "eBoard_remote_control:0805-NO" H 10700 8200 50  0001 C CNN
+F 2 "eBoard_remote_control:C0603" H 10700 8200 50  0001 C CNN
 F 3 "" H 10700 8200 50  0001 C CNN
 	1    10700 8200
@@
 F 0 "DIS1" H 14900 1650 59  0000 C CNN
 F 1 "OLED" H 15070 2000 59  0000 C CNN
-F 2 "Connector_PinHeader_2.54mm:PinHeader_1x04_P2.54mm_Vertical" H 14900 1900 50  0001 C CNN
+F 2 "eBoard_remote_control:OLED" H 14900 1900 50  0001 C CNN
 F 3 "" H 14900 1900 50  0001 C CNN
 	1    14900 1900
@@
 Text Label 2400 3900 0    50   ~ 0
 VBB
-$Comp
-L Connector:Conn_01x05_Male J1
-U 1 1 5BDA5CA2
-P 11400 4300
-F 0 "J1" H 11508 4681 50  0000 C CNN
-F 1 "SWDIO_conn" H 11508 4590 50  0000 C CNN
-F 2 "Connector_PinHeader_2.54mm:PinHeader_1x05_P2.54mm_Vertical" H 11400 4300 50  0001 C CNN
-F 3 "~" H 11400 4300 50  0001 C CNN
-	1    11400 4300
-	1    0    0    -1
-$EndComp
-Wire Wire Line
-	11800 4100 11600 4100
-Wire Wire Line
-	11800 4200 11600 4200
-Wire Wire Line
-	11800 4300 11600 4300
-Wire Wire Line
-	11800 4400 11600 4400
-Wire Wire Line
-	11800 4500 11600 4500
-Text Label 11800 4100 0    50   ~ 0
+Text Label 11300 4400 0    50   ~ 0
 GND
-Text Label 11800 4200 0    50   ~ 0
+Text Label 11300 3900 0    50   ~ 0
 3.3V
-Text Label 11800 4300 0    50   ~ 0
+Text Label 12200 3900 0    50   ~ 0
 SWDIO
-Text Label 11800 4400 0    50   ~ 0
+Text Label 12200 4000 0    50   ~ 0
 SWCLK
-Text Label 11800 4500 0    50   ~ 0
+Text Label 12200 4300 0    50   ~ 0
 RESET
 Wire Wire Line
@@
 Wire Wire Line
 	12300 1900 14000 1900
+$Comp
+L eBoard_remote_control-eagle-import:CAP_CERAMIC0603_NO C9
+U 1 1 5C35532F
+P 13800 7200
+F 0 "C9" V 13585 7250 50  0000 C CNN
+F 1 "0.1uF" V 13676 7250 50  0000 C CNN
+F 2 "eBoard_remote_control:C0603" H 13800 7200 50  0001 C CNN
+F 3 "" H 13800 7200 50  0001 C CNN
+	1    13800 7200
+	0    1    1    0
+$EndComp
+$Comp
+L eBoard_remote_control-eagle-import:SOLDERJUMPERCLOSED SJ2
+U 1 1 5C35574F
+P 14500 7200
+F 0 "SJ2" H 14500 7446 59  0000 C CNN
+F 1 "BAT" H 14500 7341 59  0000 C CNN
+F 2 "Adafruit nRF52 Bluefruit Feather rev G:SOLDERJUMPER_CLOSEDWIRE" H 14500 7200 50  0001 C CNN
+F 3 "" H 14500 7200 50  0001 C CNN
+	1    14500 7200
+	1    0    0    -1
+$EndComp
+$Comp
+L eBoard_remote_control-eagle-import:DIODESOD-323 D4
+U 1 1 5C355C1A
+P 15100 6800
+F 0 "D4" V 15140 6722 42  0000 R CNN
+F 1 "1n4148" V 15061 6722 42  0000 R CNN
+F 2 "Adafruit nRF52 Bluefruit Feather rev G:SOD-323" H 15100 6800 50  0001 C CNN
+F 3 "" H 15100 6800 50  0001 C CNN
+	1    15100 6800
+	0    -1   -1   0
+$EndComp
+Wire Wire Line
+	14000 7200 14300 7200
+Wire Wire Line
+	13500 7200 13700 7200
+Text Label 13500 7200 0    50   ~ 0
+DTR
+Wire Wire Line
+	15100 6900 15100 7200
+Text Label 14900 7200 0    50   ~ 0
+RESET
+Wire Wire Line
+	15100 6400 15100 6500
+$Comp
+L eBoard_remote_control-eagle-import:3.3V #U$0102
+U 1 0 5C37D9A8
+P 15100 6300
+F 0 "#U$0102" H 15100 6300 50  0001 C CNN
+F 1 "3.3V" H 15040 6340 42  0000 L BNN
+F 2 "" H 15100 6300 50  0001 C CNN
+F 3 "" H 15100 6300 50  0001 C CNN
+	1    15100 6300
+	1    0    0    -1
+$EndComp
+$Comp
+L eBoard_remote_control-eagle-import:RESISTOR0805_NOOUTLINE R2
+U 1 1 5C37E6BF
+P 14800 6700
+F 0 "R2" V 14762 6778 50  0000 L CNN
+F 1 "10K" V 14846 6778 40  0000 L CNB
+F 2 "eBoard_remote_control:0603-NO" H 14800 6700 50  0001 C CNN
+F 3 "" H 14800 6700 50  0001 C CNN
+	1    14800 6700
+	0    1    1    0
+$EndComp
+Connection ~ 15100 6500
+Wire Wire Line
+	15100 6500 15100 6700
+Wire Wire Line
+	14700 7200 14800 7200
+Wire Wire Line
+	14800 6500 15100 6500
+Wire Wire Line
+	14800 6900 14800 7200
+Connection ~ 14800 7200
+Wire Wire Line
+	14800 7200 15100 7200
+$Comp
+L Adafruit_nRF52_Bluefruit_Feather_rev_G-cache:Adafruit_nRF52_Bluefruit_Feather_rev_G-eagle-import_JTAG-CORTEXBOXPOSTS J1
+U 1 1 5C356BF2
+P 11700 4100
+F 0 "J1" H 11700 4547 42  0000 C CNN
+F 1 "SWDIO_conn" H 11700 4468 42  0000 C CNN
+F 2 "Connector_PinHeader_1.27mm:PinHeader_2x05_P1.27mm_Vertical_SMD" H 11700 4100 50  0000 C CNN
+F 3 "" H 11700 4100 50  0001 C CNN
+	1    11700 4100
+	1    0    0    -1
+$EndComp
+Wire Wire Line
+	12200 3900 12000 3900
+Wire Wire Line
+	12200 4000 12000 4000
+Wire Wire Line
+	12200 4100 12000 4100
+Wire Wire Line
+	12200 4200 12000 4200
+Wire Wire Line
+	12200 4300 12000 4300
+Wire Wire Line
+	11400 4000 11300 4000
+Wire Wire Line
+	11300 4000 11300 4100
+Wire Wire Line
+	11300 4100 11400 4100
+Wire Wire Line
+	11300 4100 11300 4200
+Wire Wire Line
+	11300 4200 11400 4200
+Connection ~ 11300 4100
+Wire Wire Line
+	11300 4200 11300 4300
+Wire Wire Line
+	11300 4300 11400 4300
+Connection ~ 11300 4200
+Wire Wire Line
+	11300 4400 11300 4300
+Connection ~ 11300 4300
+Wire Wire Line
+	11300 3900 11400 3900
 $EndSCHEMATC

Commit message: V2.1
Changed lines of the file:
@@
 F 0 "J1" H 11700 4547 42  0000 C CNN
 F 1 "SWDIO_conn" H 11700 4468 42  0000 C CNN
-F 2 "Connector_PinHeader_1.27mm:PinHeader_2x05_P1.27mm_Vertical_SMD" H 11700 4100 50  0000 C CNN
+F 2 "Connector_PinHeader_1.27mm:PinHeader_2x05_P1.27mm_Vertical_SMD" H 11600 4700 50  0000 C CNN
 F 3 "" H 11700 4100 50  0001 C CNN
 	1    11700 4100
@@
 Wire Wire Line
 	11300 3900 11400 3900
+Text Label 12200 4100 0    50   ~ 0
+SWO
 $EndSCHEMATC

Commit message: this
Parts:
- removed DIS1: OLED, eBoard_remote_control:OLED, symbol eBoard_remote_control-eagle-import:OLED
- added U8: SSD1306, eBoard_remote_control:SSD1306_OLED-0.91-128x32, symbol SSD1306_OLED-0.91-128x32:SSD1306
Connections:
- wire segments 188 -> 183
Changed lines of the file:
@@
-GND
-Wire Wire Line
-	14000 2000 13900 2000
-Wire Wire Line
-	13900 2000 13900 2400
-Text Label 14000 2000 0    10   ~ 0
 GND
 Wire Wire Line
@@
 Text Label 14100 3800 1    50   ~ 0
 3.3V
-Text Label 12300 1900 2    50   ~ 0
-3.3V
 Wire Wire Line
 	3100 7300 3000 7300
 Text Label 3000 7300 2    50   ~ 0
 SDA
-Text Label 12300 1700 2    50   ~ 0
-SDA
 Wire Wire Line
 	3100 7400 3000 7400
 Text Label 3000 7400 2    50   ~ 0
-SCL
-Text Label 12300 1800 2    50   ~ 0
 SCL
 Wire Wire Line
@@
 	1    15400 4300
 	0    1    1    0
-$EndComp
-$Comp
-L eBoard_remote_control-eagle-import:OLED DIS1
-U 1 0 E925ABD7
-P 14900 1900
-F 0 "DIS1" H 14900 1650 59  0000 C CNN
-F 1 "OLED" H 15070 2000 59  0000 C CNN
-F 2 "eBoard_remote_control:OLED" H 14900 1900 50  0001 C CNN
-F 3 "" H 14900 1900 50  0001 C CNN
-	1    14900 1900
-	1    0    0    -1
-$EndComp
-$Comp
-L eBoard_remote_control-eagle-import:GND #GND04
-U 1 0 12C122FD
-P 13900 2500
-F 0 "#GND04" H 13900 2500 50  0001 C CNN
-F 1 "GND" H 13800 2400 59  0000 L BNN
-F 2 "" H 13900 2500 50  0001 C CNN
-F 3 "" H 13900 2500 50  0001 C CNN
-	1    13900 2500
-	1    0    0    -1
 $EndComp
 $Comp
@@
 Wire Wire Line
 	9600 3400 9600 3800
-Wire Wire Line
-	12300 1800 14000 1800
-Wire Wire Line
-	12300 1700 14000 1700
-Wire Wire Line
-	12300 1900 14000 1900
 $Comp
 L eBoard_remote_control-eagle-import:CAP_CERAMIC0603_NO C9
@@
 Text Label 12200 4100 0    50   ~ 0
 SWO
+$Comp
+L SSD1306_OLED-0.91-128x32:SSD1306 U8
+U 1 1 5CC03FF3
+P 13900 2350
+F 0 "U8" H 13900 3187 60  0000 C CNN
+F 1 "SSD1306" H 13900 3081 60  0000 C CNN
+F 2 "eBoard_remote_control:SSD1306_OLED-0.91-128x32" H 13900 2350 60  0001 C CNN
+F 3 "" H 13900 2350 60  0001 C CNN
+	1    13900 2350
+	1    0    0    -1
+$EndComp
 $EndSCHEMATC

Commit message: this
Parts:
- added C?: 10µF, eBoard_remote_control:C0603, symbol eBoard_remote_control-eagle-import:C"
- added C?: 100n, eBoard_remote_control:C0603, symbol eBoard_remote_control-eagle-import:C"
- added R1: 1K, eBoard_remote_control:0603-NO, symbol eBoard_remote_control-eagle-import:RESISTOR_0603_NOOUT
Connections:
- net DTR: now also R1.2
- net GND: now also C?.2, C?.2, R1.1
- new net: C?.1, C?.1
Other:
- moved on the sheet: U8
Changed lines of the file:
@@
 3.3V
-Wire Wire Line
-	8300 1800 8300 1600
-Wire Wire Line
-	8300 1600 8300 1400
 Wire Wire Line
 	7300 1900 7300 1600
@@
 Text Label 8300 1400 1    50   ~ 0
 3.3V
-Connection ~ 8300 1600
 Connection ~ 7600 1600
 Wire Wire Line
@@
 Text Notes 13200 3400 0    59   ~ 0
 Trigger
-Text Notes 13800 1200 0    59   ~ 0
+Text Notes 13600 950  0    59   ~ 0
 OLED Display
 Wire Notes Line
@@
 Wire Wire Line
 	14000 7200 14300 7200
-Wire Wire Line
-	13500 7200 13700 7200
-Text Label 13500 7200 0    50   ~ 0
+Text Label 13350 7200 0    50   ~ 0
 DTR
 Wire Wire Line
@@
 L SSD1306_OLED-0.91-128x32:SSD1306 U8
 U 1 1 5CC03FF3
-P 13900 2350
-F 0 "U8" H 13900 3187 60  0000 C CNN
-F 1 "SSD1306" H 13900 3081 60  0000 C CNN
-F 2 "eBoard_remote_control:SSD1306_OLED-0.91-128x32" H 13900 2350 60  0001 C CNN
-F 3 "" H 13900 2350 60  0001 C CNN
-	1    13900 2350
-	1    0    0    -1
-$EndComp
+P 15050 2150
+F 0 "U8" H 15050 2987 60  0000 C CNN
+F 1 "SSD1306" H 15050 2881 60  0000 C CNN
+F 2 "eBoard_remote_control:SSD1306_OLED-0.91-128x32" H 15050 2150 60  0001 C CNN
+F 3 "" H 15050 2150 60  0001 C CNN
+	1    15050 2150
+	0    1    1    0
+$EndComp
+$Comp
+L eBoard_remote_control-eagle-import:RESISTOR_0603_NOOUT R1
+U 1 0 5CBFBD28
+P 13650 7500
+F 0 "R1" H 13650 7600 50  0000 C CNN
+F 1 "1K" H 13650 7500 40  0000 C CNB
+F 2 "eBoard_remote_control:0603-NO" H 13650 7500 50  0001 C CNN
+F 3 "" H 13650 7500 50  0001 C CNN
+	1    13650 7500
+	0    -1   -1   0
+$EndComp
+Wire Wire Line
+	13350 7200 13650 7200
+Wire Wire Line
+	13650 7300 13650 7200
+Connection ~ 13650 7200
+Wire Wire Line
+	13650 7200 13700 7200
+$Comp
+L power:GND #PWR0101
+U 1 1 5CC257DF
+P 13650 7900
+F 0 "#PWR0101" H 13650 7650 50  0001 C CNN
+F 1 "GND" H 13655 7727 50  0000 C CNN
+F 2 "" H 13650 7900 50  0001 C CNN
+F 3 "" H 13650 7900 50  0001 C CNN
+	1    13650 7900
+	1    0    0    -1
+$EndComp
+Wire Wire Line
+	13650 7700 13650 7900
+Connection ~ 8300 1600
+Wire Wire Line
+	8300 1600 8300 1400
+Wire Wire Line
+	8300 1800 8300 1600
+Wire Wire Line
+	8600 4200 8600 4300
+Text Label 8600 4200 0    10   ~ 0
+GND
+Wire Wire Line
+	8900 4200 8900 4300
+Text Label 8900 4200 0    10   ~ 0
+GND
+Wire Wire Line
+	8600 3900 8600 3600
+Wire Wire Line
+	8600 3600 8900 3600
+Wire Wire Line
+	8900 3600 9600 3600
+Wire Wire Line
+	8900 3900 8900 3600
+Connection ~ 8900 3600
+$Comp
+L eBoard_remote_control-eagle-import:C" C?
+U 1 0 5CC3F841
+P 8600 4000
+F 0 "C?" V 8509 4049 59  0000 C CNN
+F 1 "10µF" V 8690 4049 59  0000 C CNN
+F 2 "eBoard_remote_control:C0603" H 8600 4000 50  0001 C CNN
+F 3 "" H 8600 4000 50  0001 C CNN
+	1    8600 4000
+	1    0    0    -1
+$EndComp
+$Comp
+L eBoard_remote_control-eagle-import:GND #GND?
+U 1 0 5CC3F847
+P 8600 4400
+F 0 "#GND?" H 8600 4400 50  0001 C CNN
+F 1 "GND" H 8500 4300 59  0000 L BNN
+F 2 "" H 8600 4400 50  0001 C CNN
+F 3 "" H 8600 4400 50  0001 C CNN
+	1    8600 4400
+	1    0    0    -1
+$EndComp
+$Comp
+L eBoard_remote_control-eagle-import:C" C?
+U 1 0 5CC3F84D
+P 8900 4000
+F 0 "C?" V 8809 4049 59  0000 C CNN
+F 1 "100n" V 8990 4049 59  0000 C CNN
+F 2 "eBoard_remote_control:C0603" H 8900 4000 50  0001 C CNN
+F 3 "" H 8900 4000 50  0001 C CNN
+	1    8900 4000
+	1    0    0    -1
+$EndComp
+$Comp
+L eBoard_remote_control-eagle-import:GND #GND?
+U 1 0 5CC3F853
+P 8900 4400
+F 0 "#GND?" H 8900 4400 50  0001 C CNN
+F 1 "GND" H 8800 4300 59  0000 L BNN
+F 2 "" H 8900 4400 50  0001 C CNN
+F 3 "" H 8900 4400 50  0001 C CNN
+	1    8900 4400
+	1    0    0    -1
+$EndComp

Commit message: this
Parts:
- removed P1: USB, eBoard_remote_control:USB-MICRO-B, symbol eBoard_remote_control-eagle-import:USB
- added J2: 105450-0101, eBoard_remote_control:105450-0101, symbol 2019-04-23_17-32-18:105450-0101
- added X?: JSTPH, eBoard_remote_control:JSTPH2, symbol eBoard_remote_control-eagle-import:CON_JST_PH_2PIN
- gave numbers to parts that had none: 2
Connections:
- net GND: now also J2.A1, J2.A12, J2.B1, J2.B12, X?.1
- net USBD+: now also J2.A6, J2.B6
- net USBD-: now also J2.A7, J2.B7
- net VBAT: now also X?.2
- net VBUS: now also J2.A4, J2.A9, J2.B4, J2.B9
Other:
- moved on the sheet: C17
Changed lines of the file:
@@
-GND
-Wire Wire Line
-	8300 7800 8600 7800
-Wire Wire Line
-	8600 7800 8600 8300
-Wire Wire Line
-	8300 7600 8600 7600
-Wire Wire Line
-	8600 7600 8600 7800
-Connection ~ 8600 7800
-Text Label 8300 7800 0    10   ~ 0
-GND
-Wire Wire Line
-	9200 7800 9200 8300
-Text Label 9200 7800 0    10   ~ 0
 GND
 Wire Wire Line
@@
 VBUS
 Wire Wire Line
-	8300 6800 9200 6800
-Wire Wire Line
-	9200 6800 9400 6800
-Wire Wire Line
-	9200 7500 9200 6800
-Text Label 9400 6800 0    50   ~ 0
-VBUS
-Connection ~ 9200 6800
-Wire Wire Line
 	4900 4000 4900 4400
 Text Label 4900 4000 0    10   ~ 0
@@
 USBD+
 Wire Wire Line
-	8300 7200 8600 7200
-Text Label 8600 7200 0    50   ~ 0
-USBD+
-Wire Wire Line
 	10900 7700 11000 7700
 Text Label 10900 7700 2    50   ~ 0
-USBD-
-Wire Wire Line
-	8300 7000 8600 7000
-Text Label 8600 7000 0    50   ~ 0
 USBD-
 Wire Wire Line
@@
 $EndComp
 $Comp
-L eBoard_remote_control-eagle-import:USB P1
-U 1 0 24F1395A
-P 7900 7100
-F 0 "P1" H 7500 6800 42  0000 L BNN
-F 1 "USB" H 7900 7100 50  0001 C CNN
-F 2 "eBoard_remote_control:USB-MICRO-B" H 7900 7100 50  0001 C CNN
-F 3 "" H 7900 7100 50  0001 C CNN
-	1    7900 7100
-	0    1    1    0
-$EndComp
-$Comp
-L eBoard_remote_control-eagle-import:GND #U$013
-U 1 0 33430DC8
-P 8600 8400
-F 0 "#U$013" H 8600 8400 50  0001 C CNN
-F 1 "GND" H 8540 8300 59  0000 L BNN
-F 2 "" H 8600 8400 50  0001 C CNN
-F 3 "" H 8600 8400 50  0001 C CNN
-	1    8600 8400
-	1    0    0    -1
-$EndComp
-$Comp
 L eBoard_remote_control-eagle-import:C" C17
 U 1 0 A18871AA
-P 9200 7600
-F 0 "C17" V 9109 7649 59  0000 C CNN
-F 1 "10µF" V 9290 7649 59  0000 C CNN
-F 2 "eBoard_remote_control:C0603" H 9200 7600 50  0001 C CNN
-F 3 "" H 9200 7600 50  0001 C CNN
-	1    9200 7600
-	1    0    0    -1
-$EndComp
-$Comp
-L eBoard_remote_control-eagle-import:GND #GND07
-U 1 0 C2693486
-P 9200 8400
-F 0 "#GND07" H 9200 8400 50  0001 C CNN
-F 1 "GND" H 9100 8300 59  0000 L BNN
-F 2 "" H 9200 8400 50  0001 C CNN
-F 3 "" H 9200 8400 50  0001 C CNN
-	1    9200 8400
-	1    0    0    -1
+P 8700 6900
+F 0 "C17" V 8609 6949 59  0000 C CNN
+F 1 "10µF" V 8790 6949 59  0000 C CNN
+F 2 "eBoard_remote_control:C0603" H 8700 6900 50  0001 C CNN
+F 3 "" H 8700 6900 50  0001 C CNN
+	1    8700 6900
+	-1   0    0    1
 $EndComp
 $Comp
@@
 	1200 10500 1200 5500
 Wire Notes Line
-	7100 9100 15900 9100
+	15850 9450 7050 9450
 Wire Notes Line
 	15900 9100 15900 5500
@@
 Connection ~ 8900 3600
 $Comp
-L eBoard_remote_control-eagle-import:C" C?
+L eBoard_remote_control-eagle-import:C" C11
 U 1 0 5CC3F841
 P 8600 4000
-F 0 "C?" V 8509 4049 59  0000 C CNN
+F 0 "C11" V 8509 4049 59  0000 C CNN
 F 1 "10µF" V 8690 4049 59  0000 C CNN
 F 2 "eBoard_remote_control:C0603" H 8600 4000 50  0001 C CNN
@@
 $EndComp
 $Comp
-L eBoard_remote_control-eagle-import:GND #GND?
+L eBoard_remote_control-eagle-import:GND #GND0102
 U 1 0 5CC3F847
 P 8600 4400
-F 0 "#GND?" H 8600 4400 50  0001 C CNN
+F 0 "#GND0102" H 8600 4400 50  0001 C CNN
 F 1 "GND" H 8500 4300 59  0000 L BNN
 F 2 "" H 8600 4400 50  0001 C CNN
@@
 $EndComp
 $Comp
-L eBoard_remote_control-eagle-import:C" C?
+L eBoard_remote_control-eagle-import:C" C13
 U 1 0 5CC3F84D
 P 8900 4000
-F 0 "C?" V 8809 4049 59  0000 C CNN
+F 0 "C13" V 8809 4049 59  0000 C CNN
 F 1 "100n" V 8990 4049 59  0000 C CNN
 F 2 "eBoard_remote_control:C0603" H 8900 4000 50  0001 C CNN
@@
 $EndComp
 $Comp
-L eBoard_remote_control-eagle-import:GND #GND?
+L eBoard_remote_control-eagle-import:GND #GND0103
 U 1 0 5CC3F853
 P 8900 4400
-F 0 "#GND?" H 8900 4400 50  0001 C CNN
+F 0 "#GND0103" H 8900 4400 50  0001 C CNN
 F 1 "GND" H 8800 4300 59  0000 L BNN
 F 2 "" H 8900 4400 50  0001 C CNN
@@
 	1    0    0    -1
 $EndComp
+$Comp
+L 2019-04-23_17-32-18:105450-0101 J2
+U 1 1 5CC48FA5
+P 8050 9000
+F 0 "J2" H 8578 7903 60  0000 L CNN
+F 1 "105450-0101" H 8578 7797 60  0000 L CNN
+F 2 "eBoard_remote_control:105450-0101" H 8450 7740 60  0001 C CNN
+F 3 "" H 8050 9000 60  0000 C CNN
+	1    8050 9000
+	-1   0    0    1
+$EndComp
+$Comp
+L power:GND #PWR0102
+U 1 1 5CC5E143
+P 8950 9200
+F 0 "#PWR0102" H 8950 8950 50  0001 C CNN
+F 1 "GND" H 8955 9027 50  0000 C CNN
+F 2 "" H 8950 9200 50  0001 C CNN
+F 3 "" H 8950 9200 50  0001 C CNN
+	1    8950 9200
+	1    0    0    -1
+$EndComp
+Wire Wire Line
+	8050 9000 8950 9000
+Wire Wire Line
+	8950 9000 8950 7900
+Wire Wire Line
+	8050 6700 8700 6700
+Wire Wire Line
+	8950 9000 8950 9200
+Wire Wire Line
+	8050 7800 8950 7800
+Connection ~ 8950 7800
+Wire Wire Line
+	8950 7800 8950 6700
+Wire Wire Line
+	8050 7900 8950 7900
+Connection ~ 8950 7900
+Wire Wire Line
+	8950 7900 8950 7800
+Wire Wire Line
+	8050 8700 8700 8700
+Wire Wire Line
+	8400 7000 8400 6600
+Wire Wire Line
+	8050 7000 8400 7000
+Wire Wire Line
+	8700 7000 8700 7500
+Wire Wire Line
+	8050 8200 8700 8200
+Connection ~ 8700 8200
+Wire Wire Line
+	8700 8200 8700 8700
+Wire Wire Line
+	8050 7500 8700 7500
+Connection ~ 8700 7500
+Wire Wire Line
+	8700 7500 8700 8200
+Text Label 8400 6600 0    50   ~ 0
+VBUS
+Connection ~ 8700 7000
+Connection ~ 8700 6700
+Wire Wire Line
+	8700 6700 8950 6700
+Wire Wire Line
+	8050 8500 8300 8500
+Wire Wire Line
+	8050 8400 8300 8400
+Wire Wire Line
+	8050 7200 8350 7200
+Wire Wire Line
+	8050 7300 8350 7300
+Text GLabel 8300 8500 2    50   Input ~ 0
+USBD+
+Text GLabel 8300 8400 2    50   Input ~ 0
+USBD-
+Text GLabel 8350 7200 2    50   Input ~ 0
+USBD-
+Text GLabel 8350 7300 2    50   Input ~ 0
+USBD+
+Connection ~ 8950 9000
+Connection ~ 8400 7000
+Wire Wire Line
+	8400 7000 8700 7000
+Wire Wire Line
+	4500 4900 4500 4500
+Text Label 4500 4900 0    10   ~ 0
+GND
+Wire Wire Line
+	4500 4000 4500 4400
+Text Label 4500 4000 0    10   ~ 0
+VBAT
+$Comp
+L eBoard_remote_control-eagle-import:CON_JST_PH_2PIN X?
+U 1 0 5CD5CAD6
+P 4400 4400
+F 0 "X?" H 4150 4625 59  0000 L BNN
+F 1 "JSTPH" H 4150 4200 59  0000 L BNN
+F 2 "eBoard_remote_control:JSTPH2" H 4400 4400 50  0001 C CNN
+F 3 "" H 4400 4400 50  0001 C CNN
+	1    4400 4400
+	-1   0    0    1
+$EndComp
+$Comp
+L eBoard_remote_control-eagle-import:VBAT #U$?
+U 1 0 5CD5CADC
+P 4500 3900
+F 0 "#U$?" H 4500 3900 50  0001 C CNN
+F 1 "VBAT" H 4440 3940 42  0000 L BNN
+F 2 "" H 4500 3900 50  0001 C CNN
+F 3 "" H 4500 3900 50  0001 C CNN
+	1    4500 3900
+	1    0    0    -1
+$EndComp
+$Comp
+L eBoard_remote_control-eagle-import:GND #U$?
+U 1 0 5CD5CAE2
+P 4500 5000
+F 0 "#U$?" H 4500 5000 50  0001 C CNN
+F 1 "GND" H 4440 4900 59  0000 L BNN
+F 2 "" H 4500 5000 50  0001 C CNN
+F 3 "" H 4500 5000 50  0001 C CNN
+	1    4500 5000
+	1    0    0    -1
+$EndComp
