File: eBoard_remote_control/eBoard_remote_control.sch (KiCad schematic (older format))
At the start: 46 parts, among them J1 SWDIO_conn, J2 105450-0101, U1 MDBT42, U2 AP2112(3.3V), U3 MCP73831T-2ACI/OT, U4 CP2104, U5 AH49ENTR-G1, U6 AH49ENTR-G1, U7 AH49ENTR-G1, U8 SSD1306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

Commit message: oled schem
Parts:
- removed R10: 1K, eBoard_remote_control:0603-NO, symbol eBoard_remote_control-eagle-import:RESISTOR_0603_NOOUT
- added C15: 100nF, eBoard_remote_control:C0603, symbol eBoard_remote_control-eagle-import:C"
- added C18, C19, C22, C25, C26: 1uF, eBoard_remote_control:C0603, symbol eBoard_remote_control-eagle-import:C"
- added C23, C24: 10uF, eBoard_remote_control:C0603, symbol eBoard_remote_control-eagle-import:C"
- added R11: 390k, eBoard_remote_control:0603-NO, symbol eBoard_remote_control-eagle-import:RESISTOR_0603_NOOUT
- added R7: 10K, eBoard_remote_control:0603-NO, symbol eBoard_remote_control-eagle-import:RESISTOR_0603_NOOUT
- C13, C16, C21: value 100n -> 100nF
- gave numbers to parts that had none: 1
Connections:
- net 3.3V: now also C15.1
- net GND: now also U8.7 (VSS), C15.2, C22.1, C23.1, C24.1, R11.2
- net SCL: now also U8.10 (SCL)
- net SDA: now also U8.11 (SDA)
- net at U8.1 (C2P): now also C18.1
- net at U8.12 (IREF): now also R11.1
- net at U8.13 (VCOMH): now also C23.2
- net at U8.14 (VCC): now also C24.2
- net at U8.2 (C2N): now also C18.2
- net at U8.3 (C1P): now also C19.1
- net at U8.4 (C1N): now also C19.2
- net 3V3: now reaches U8.5 (VDDB)
- net 3V3: now also U8.8 (VDD), R7.2
- net at U8.6 (NC): now also C22.2
- net at U8.9 (~RES): now also R7.1
Other:
- moved on the sheet: U8

Commit message: started Layout V3
Parts:
- removed C25, C26: 1uF, eBoard_remote_control:C0603, symbol eBoard_remote_control-eagle-import:C"
Connections:
- net 3.3V: no longer U6.1 (VCC)
- net 3V3: now also C11.1, C13.1, U6.1 (VCC)
Changed lines of the file:
@@
 Text Label 9600 4800 0    10   ~ 0
 GND
-Text Label 9600 3400 1    50   ~ 0
-3.3V
 Wire Wire Line
 	10200 4300 10300 4300
@@
 Text Label 12200 4300 0    50   ~ 0
 RESET
-Wire Wire Line
-	9600 3400 9600 3800
 $Comp
 L eBoard_remote_control-eagle-import:CAP_CERAMIC0603_NO C9
@@
 Text Label 8900 4200 0    10   ~ 0
 GND
-Wire Wire Line
-	8600 3900 8600 3600
-Wire Wire Line
-	8600 3600 8900 3600
-Wire Wire Line
-	8900 3600 9600 3600
-Wire Wire Line
-	8900 3900 8900 3600
-Connection ~ 8900 3600
 $Comp
 L eBoard_remote_control-eagle-import:C" C11
@@
 	13400 1750 13400 1850
 $Comp
-L eBoard_remote_control-eagle-import:C" C26
-U 1 0 5CDED170
-P 26850 16950
-F 0 "C26" V 26759 16999 59  0000 C CNN
-F 1 "1uF" V 26940 16999 59  0000 C CNN
-F 2 "eBoard_remote_control:C0603" H 26850 16950 50  0001 C CNN
-F 3 "" H 26850 16950 50  0001 C CNN
-	1    26850 16950
-	0    -1   -1   0
-$EndComp
-$Comp
-L eBoard_remote_control-eagle-import:C" C25
-U 1 0 5CDFA6D1
-P 26500 17650
-F 0 "C25" V 26409 17699 59  0000 C CNN
-F 1 "1uF" V 26590 17699 59  0000 C CNN
-F 2 "eBoard_remote_control:C0603" H 26500 17650 50  0001 C CNN
-F 3 "" H 26500 17650 50  0001 C CNN
-	1    26500 17650
-	0    -1   -1   0
-$EndComp
-$Comp
 L eBoard_remote_control-eagle-import:C" C22
 U 1 0 5CE07423
@@
 Wire Wire Line
 	13400 4600 14300 4600
+Wire Wire Line
+	9600 3400 9600 3550
+Wire Wire Line
+	8900 3900 8900 3550
+Wire Wire Line
+	8900 3550 9600 3550
+Wire Wire Line
+	8900 3550 8600 3550
+Wire Wire Line
+	8600 3550 8600 3900
+Connection ~ 8900 3550
+Text Label 9600 3400 1    50   ~ 0
+3V3
+Wire Wire Line
+	9600 3550 9600 3800
+Connection ~ 9600 3550
 $EndSCHEMATC

Commit message: added rgb led V3
Parts:
- added D1: LED_ARGB, LED_SMD:LED_Avago_PLCC4_3.2x2.8mm_CW, symbol Device:LED_ARGB
Connections:
- net 3V3: now also D1.1 (A)
- net at U1.31 (P0.17): now also D1.3 (GK)
- net at U1.33 (P0.19): now also D1.2 (RK)
Changed lines of the file:
@@
 	9600 3550 9600 3800
 Connection ~ 9600 3550
+$Comp
+L Device:LED_ARGB D1
+U 1 1 5CCBD6F3
+P 6000 8550
+F 0 "D1" H 6000 9047 50  0000 C CNN
+F 1 "LED_ARGB" H 6000 8956 50  0000 C CNN
+F 2 "LED_SMD:LED_Avago_PLCC4_3.2x2.8mm_CW" H 6000 8500 50  0001 C CNN
+F 3 "~" H 6000 8500 50  0001 C CNN
+	1    6000 8550
+	1    0    0    -1
+$EndComp
+Wire Wire Line
+	4900 7700 5500 7700
+Wire Wire Line
+	5500 7700 5500 8550
+Wire Wire Line
+	5500 8550 5800 8550
+Wire Wire Line
+	5800 8350 5650 8350
+Wire Wire Line
+	5650 8350 5650 7500
+Wire Wire Line
+	5650 7500 4900 7500
+Wire Wire Line
+	6450 8550 6200 8550
+Text GLabel 6450 8550 2    50   Input ~ 0
+3V3
 $EndSCHEMATC
