File: eBoard_remote_control/eBoard_remote_control.kicad_pcb (KiCad board)
At the start: 2 copper layers, 34 x 99.9 mm, 53 parts, among them J1 SWDIO_conn, J2 105450-0101, U1 MDBT42, U2 AP2112(3.3V), U3 MCP73831T-2ACI/OT, U4 CP2104, U5 AH49ENTR-G1, U6 AH49ENTR-G1, U7 AH49ENTR-G1, U8 SSD1306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

Commit message: added rgb led V3
Parts:
- added D1: LED_ARGB, LED_SMD:LED_Avago_PLCC4_3.2x2.8mm_CW, F.Cu at (198.8, 135.3)
Changed lines of the file:
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@@
     (tracks 330)
     (zones 0)
-    (modules 53)
-    (nets 43)
+    (modules 54)
+    (nets 47)
   )
   (page A4)
@@
   (net 41 SDA)
   (net 42 SCL)
+  (net 43 "Net-(D1-Pad4)")
+  (net 44 "Net-(D1-Pad3)")
+  (net 45 "Net-(D1-Pad2)")
+  (net 46 "Net-(D1-Pad1)")
   (net_class Default "This is the default net class."
     (clearance 0.2)
@@
     (add_net "Net-(C9-Pad1)")
     (add_net "Net-(CHG1-PadC)")
+    (add_net "Net-(D1-Pad1)")
+    (add_net "Net-(D1-Pad2)")
+    (add_net "Net-(D1-Pad3)")
+    (add_net "Net-(D1-Pad4)")
     (add_net "Net-(L2-Pad2)")
     (add_net "Net-(R11-Pad1)")
@@
     (uvia_drill 0.1)
   )
+  (module LED_SMD:LED_Avago_PLCC4_3.2x2.8mm_CW (layer Top)
+    (at 198.75 135.35 90)
+    (descr https://docs.broadcom.com/docs/AV02-4186EN)
+    (tags "LED Avago PLCC-4 ASMB-MTB0-0A3A2")
+    (attr smd)
+    (fp_text reference D1 (at 0 -2.65 90) (layer F.SilkS)
+      (effects (font (size 1 1) (thickness 0.15)))
+    )
+    (fp_text value LED_ARGB (at 0 2.65 90) (layer F.Fab)
+      (effects (font (size 1 1) (thickness 0.15)))
+    )
+    (fp_circle (center 0 0) (end 1.12 0) (layer F.Fab) (width 0.1))
+    (fp_line (start 2.5 1.65) (end -2.5 1.65) (layer F.CrtYd) (width 0.05))
+    (fp_line (start 2.5 1.65) (end 2.5 -1.65) (layer F.CrtYd) (width 0.05))
+    (fp_line (start -2.5 -1.65) (end -2.5 1.65) (layer F.CrtYd) (width 0.05))
+    (fp_line (start -2.5 -1.65) (end 2.5 -1.65) (layer F.CrtYd) (width 0.05))
+    (fp_line (start -1.95 1.5) (end 1.95 1.5) (layer F.SilkS) (width 0.12))
+    (fp_line (start -2.500044 -1.5) (end 1.95 -1.5) (layer F.SilkS) (width 0.12))
+    (fp_line (start -2.5 -0.7) (end -2.5 -1.5) (layer F.SilkS) (width 0.12))
+    (fp_line (start 1.6 -1.4) (end -1.6 -1.4) (layer F.Fab) (width 0.1))
+    (fp_line (start 1.6 1.4) (end 1.6 -1.4) (layer F.Fab) (width 0.1))
+    (fp_line (start -1.6 1.4) (end 1.6 1.4) (layer F.Fab) (width 0.1))
+    (fp_line (start -1.6 -1.4) (end -1.6 1.4) (layer F.Fab) (width 0.1))
+    (fp_line (start -0.6 -1.4) (end -1.6 -0.4) (layer F.Fab) (width 0.1))
+    (fp_text user %R (at 0 0 90) (layer F.Fab)
+      (effects (font (size 0.5 0.5) (thickness 0.075)))
+    )
+    (pad 4 smd rect (at -1.5 0.75 90) (size 1.5 1.1) (layers Top F.Paste F.Mask)
+      (net 43 "Net-(D1-Pad4)"))
+    (pad 3 smd rect (at 1.5 0.75 90) (size 1.5 1.1) (layers Top F.Paste F.Mask)
+      (net 44 "Net-(D1-Pad3)"))
+    (pad 2 smd rect (at 1.5 -0.75 90) (size 1.5 1.1) (layers Top F.Paste F.Mask)
+      (net 45 "Net-(D1-Pad2)"))
+    (pad 1 smd rect (at -1.5 -0.75 90) (size 1.5 1.1) (layers Top F.Paste F.Mask)
+      (net 46 "Net-(D1-Pad1)"))
+    (model ${KISYS3DMOD}/LED_SMD.3dshapes/LED_Avago_PLCC4_3.2x2.8mm_CW.wrl
+      (at (xyz 0 0 0))
+      (scale (xyz 1 1 1))
+      (rotate (xyz 0 0 0))
+    )
+  )
   (module eBoard_remote_control:105450-0101 (layer Top)

Commit message: V3
Parts:
- removed D1: LED_ARGB, LED_SMD:LED_Avago_PLCC4_3.2x2.8mm_CW
- added CHG2: BLUE, eBoard_remote_control:CHIPLED_0805_NOOUTLINE, F.Cu at (215.8, 132.9)
- added CHG3: BLUE, eBoard_remote_control:CHIPLED_0805_NOOUTLINE, F.Cu at (218.0, 132.9)
- added R10: 1K, eBoard_remote_control:0603-NO, F.Cu at (221.1, 132.1)
- added R12: 1K, eBoard_remote_control:0603-NO, F.Cu at (221.1, 134.6)
- moved C15 25.5 mm to (195.8, 117.2)
- moved C18 8.81 mm to (185.5, 87.2), turned to 180 degrees
- moved C19 8.36 mm to (185.5, 88.8), turned to 180 degrees
- moved C3 0.44 mm to (195.9, 116.0)
Routing:
- net Net-(C18-Pad2): track 12.7 -> 4.65 mm
- net Net-(C19-Pad2): track 11.1 -> 4.52 mm
- net Net-(C19-Pad1): track 9.72 -> 4.99 mm
- net Net-(C18-Pad1): track 8.75 -> 4.24 mm
- net Net-(C22-Pad2): track 9.33 -> 8.69 mm

Commit message: updated 3d modelis
Parts:
- moved R12 20.5 mm to (200.8, 132.2), turned to 90 degrees
- moved R10 18.4 mm to (202.8, 132.2), turned to 90 degrees
- moved CHG3 17.5 mm to (200.8, 135.8), turned to 180 degrees
- moved CHG2 13.3 mm to (202.8, 135.8), turned to 180 degrees
Connections:
- U1 pad 31: (no net) -> Net-(R12-Pad2)
- U1 pad 33: (no net) -> Net-(R10-Pad2)
Routing:
- net Net-(R12-Pad2): track 0.00 -> 3.94 mm
- net Net-(R10-Pad2): track 0.00 -> 3.90 mm
- net Net-(CHG3-PadA): track 0.00 -> 1.60 mm
- net Net-(CHG2-PadA): track 0.00 -> 1.60 mm

Commit message: V3
Parts:
- J2: value 105450-0101 -> USBC
- moved C2 22.5 mm to (193.0, 127.8), turned to 270 degrees
- moved C1 19.3 mm to (191.2, 125.8), turned to 270 degrees
- moved X4 13.7 mm to (191.2, 119.8), turned to 90 degrees
- moved R7 2.60 mm to (183.8, 81.4)
- moved R5 1.95 mm to (192.7, 132.9), turned to 90 degrees
- moved C22 1.63 mm to (186.6, 81.4)
- moved R9 1.57 mm to (194.2, 145.1)
- moved R11 1.14 mm to (185.2, 81.4)
- moved C3 1.01 mm to (195.0, 115.5)
- moved C15 0.86 mm to (195.0, 117.0)
- moved C10 0.40 mm to (191.0, 142.0)
- moved C6 0.27 mm to (189.5, 135.2)
- moved C8 0.20 mm to (187.5, 131.9)
Routing:
- net /A2: track 1.86 -> 53.5 mm, vias 1 -> 2
- net /A1: track 3.86 -> 50.9 mm, vias 1 -> 2
- net 3.3V: track 0.33 -> 43.6 mm, vias 0 -> 5
- net /A0: track 5.06 -> 47.4 mm, vias 1 -> 2
- net /P0.07: track 2.58 -> 37.9 mm, vias 1 -> 2
- net VBAT: track 39.5 -> 64.2 mm
- net GND: track 5.15 -> 26.5 mm, vias 4 -> 49
- net /TXD: track 11.6 -> 31.1 mm, vias 1 -> 2
- net /VBB: track 17.4 -> 35.3 mm, vias 0 -> 1
- net /RXD: track 2.87 -> 20.3 mm, vias 1 -> 0
- net VBUS: track 25.6 -> 36.9 mm
- net Net-(C2-Pad1): track 17.3 -> 11.3 mm
- net Net-(C1-Pad1): track 14.9 -> 12.2 mm
- net Net-(CHG1-PadC): track 0.00 -> 2.56 mm
- net Net-(R11-Pad1): track 8.19 -> 10.0 mm
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- added copper zone on F.Cu, net /VBB
- added copper zone on F.Cu, net 3.3V
- added copper zone on B.Cu, net GND
- added copper zone on F.Cu, net GND
Other:
- board size 34 x 99.9 mm -> 39.1 x 99.9 mm

Commit message: V3
Parts:
- J2: value USBC -> 105450-0101
- moved U7 11.1 mm to (190.1, 67.0), turned to 11.1 degrees
- moved U5 10.1 mm to (197.6, 61.4), turned to 61.8 degrees
- moved C11 3.52 mm to (188.5, 72.0), turned to 180 degrees
- moved C13 3.38 mm to (188.5, 70.5), turned to 180 degrees
- moved C16 3.09 mm to (194.5, 68.9), turned to 180 degrees
- moved C21 1.94 mm to (199.6, 65.0), turned to 180 degrees
- moved C20 1.53 mm to (194.5, 70.3), turned to 180 degrees
- moved U6 1.21 mm to (194.5, 65.0), turned to 37 degrees
- moved C14 0.43 mm to (199.6, 66.6), turned to 180 degrees
Connections:
- C11 pad 1: 3V3 -> 3.3V
- C13 pad 1: 3V3 -> 3.3V
- R7 pad 2: 3V3 -> 3.3V
- U6 pad 1: 3V3 -> 3.3V
- U8 pad 5: 3V3 -> 3.3V
- U8 pad 8: 3V3 -> 3.3V
Routing:
- net 3.3V: track 43.6 -> 156.0 mm, vias 5 -> 11
- net GND: track 26.5 -> 54.8 mm, vias 49 -> 64
- net /A0: track 47.4 -> 67.8 mm
- net /A1: track 50.9 -> 64.8 mm
- net /A2: track 53.5 -> 62.4 mm
- net 3V3: track 8.31 -> 0.00 mm
- net VBAT: track 64.2 -> 65.0 mm
Other:
- board size 39.1 x 99.9 mm -> 34 x 99.9 mm

Commit message: V3
Parts:
- moved C24 0.20 mm to (181.2, 83.2)
Routing:
- net 3.3V: track 156.0 -> 153.2 mm
- net GND: track 54.8 -> 57.5 mm, vias 64 -> 67
